File: pcb/coaster.kicad_pcb (KiCad board)
At the start: 2 copper layers, 50 x 50 mm, 21 parts, among them J1 UPDI, Q1 AO3400A, SW1 TS-1187A-B-A-B, U1 ATtiny202-SSN

Commit message: Swap LEDs to KT-0603W and drop LED resistors to 100Ω
The v0.3 board specified XL-1608UWC-04 LEDs (C965808) on the stated
rationale that they were ~3x brighter than the basic KT-0603W. The
datasheet says otherwise: XL-1608UWC-04 is 130mcd@20mA, KT-0603W is
360mcd@5mA. At the few mA a CR2016 drives through these LEDs, the
KT-0603W is ~11x brighter at the operating point — and it's a Basic
part, so no feeder fee. Drop R1-R4 150Ω→100Ω to push a little more
current now that LED efficiency, not the resistor, sets the brightness.

BOM/CPL change only; gerbers and drill stay content-identical to
v0.3.0-rc1 (component value fields don't reach the silkscreen). DRC clean.
Parts:
- L1, L2, L3, L4: value XL-1608UWC-04 -> KT-0603W
- R1, R2, R3, R4: value 150 -> 100
Changed lines of the file:
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@@
 			)
 		)
-		(property "Value" "XL-1608UWC-04"
+		(property "Value" "KT-0603W"
 			(at 0 1.43 90)
 			(layer "F.Fab")
@@
 			)
 		)
-		(property "Value" "XL-1608UWC-04"
+		(property "Value" "KT-0603W"
 			(at 0 1.43 270)
 			(layer "F.Fab")
@@
 			)
 		)
-		(property "Value" "150"
+		(property "Value" "100"
 			(at 0 1.43 90)
 			(layer "F.Fab")
@@
 			)
 		)
-		(property "Value" "150"
+		(property "Value" "100"
 			(at 0 1.43 180)
 			(layer "F.Fab")
@@
 			)
 		)
-		(property "Value" "XL-1608UWC-04"
+		(property "Value" "KT-0603W"
 			(at 0 1.43 0)
 			(layer "F.Fab")
@@
 			)
 		)
-		(property "Value" "XL-1608UWC-04"
+		(property "Value" "KT-0603W"
 			(at 0 1.43 180)
 			(layer "F.Fab")
@@
 			)
 		)
-		(property "Value" "150"
+		(property "Value" "100"
 			(at 0 1.43 0)
 			(layer "F.Fab")
@@
 			)
 		)
-		(property "Value" "150"
+		(property "Value" "100"
 			(at 0 1.43 270)
 			(layer "F.Fab")
